File: smol-FC-G474-REV-A/smol-FC-G474-REV-A.kicad_sch (KiCad schematic)
At the start: 0 parts

Commit message: Added license, and started working on schematic
Other:
- added sheet MCU (MCU.kicad_sch)
- company: (none) -> Daniel Plewa
- title: (none) -> smol-FC-G474
Changed lines of the file:
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@@
 	(generator_version "10.0")
 	(paper "A4")
+	(title_block
+		(title "smol-FC-G474")
+		(date "2026-05-24")
+		(rev "0.0.1")
+		(company "Daniel Plewa")
+		(comment 1 "GitHub: <TBA>")
+		(comment 2 "Rev A – Prototype")
+		(comment 3 "BEC 5A/2A, 10V/2A | Baro, OSD Chip and 16MB blackbox")
+		(comment 4 "Open source flight controller on STM32G4, 20x20 3.5mm hole")
+	)
+	(sheet
+		(at 127 40.64)
+		(size 50.8 86.36)
+		(exclude_from_sim no)
+		(in_bom yes)
+		(on_board yes)
+		(dnp no)
+		(fields_autoplaced yes)
+		(stroke
+			(width 0.1524)
+			(type solid)
+			(color 0 0 0 1)
+		)
+		(fill
+			(color 255 255 194 1)
+		)
+		(property "Sheetname" "MCU"
+			(at 127 39.9284 0)
+			(show_name no)
+			(do_not_autoplace no)
+			(effects
+				(font
+					(size 1.27 1.27)
+				)
+				(justify left bottom)
+			)
+		)
+		(property "Sheetfile" "MCU.kicad_sch"
+			(at 127 127.5846 0)
+			(show_name no)
+			(do_not_autoplace no)
+			(effects
+				(font
+					(size 1.27 1.27)
+				)
+				(justify left top)
+			)
+		)
+		(instances
+			(project "smol-FC-G474-REV-A"
+				(path "/650874a8-efa2-4da6-bfd2-a5dde0a9b2ac"
+					(page "2")
+				)
+			)
+		)
+	)
 	(sheet_instances
 		(path "/"
