File: smol-FC-G474-REV-A/power_supply.kicad_sch (KiCad schematic)
At the start: 30 parts, among them U10 LP5912-3.3DRV, U11 LMQ66430R5RXBR, U12 TPS2116DRL, U8 LMQ66430R5RXBR, U9 LP5912-3.3DRV

Commit message: changed size of cap on buck's
Parts:
- C29, C37: value 4.7u -> 3.3u
- C34, C39: footprint Capacitor_SMD:C_0603_1608Metric -> Capacitor_SMD:C_0402_1005Metric
Other:
- note added: "VCC CAP size changed from 0603 to 0402. Note: The LMQ66430-2EVM also uses 0402."
Changed lines of the file:
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@@
 		)
 	)
+	(text "VCC CAP size changed from 0603 to 0402.\nNote: The LMQ66430-2EVM also uses 0402."
+		(exclude_from_sim no)
+		(at 12.954 78.232 0)
+		(effects
+			(font
+				(size 0.9906 0.9906)
+				(thickness 0.1981)
+				(bold yes)
+			)
+			(justify left)
+		)
+	)
+	(text "VCC CAP size changed from 0603 to 0402.\nNote: The LMQ66430-2EVM also uses 0402."
+		(exclude_from_sim no)
+		(at 13.462 149.606 0)
+		(effects
+			(font
+				(size 0.9906 0.9906)
+				(thickness 0.1981)
+				(bold yes)
+			)
+			(justify left)
+		)
+	)
 	(text "Power MUX"
 		(exclude_from_sim no)
@@
 			)
 		)
-		(property "Footprint" "Capacitor_SMD:C_0603_1608Metric"
+		(property "Footprint" "Capacitor_SMD:C_0402_1005Metric"
 			(at 49.53 71.12 0)
 			(hide yes)
@@
 			)
 		)
-		(property "Footprint" "Capacitor_SMD:C_0603_1608Metric"
+		(property "Footprint" "Capacitor_SMD:C_0402_1005Metric"
 			(at 49.53 142.24 0)
 			(hide yes)
@@
 			)
 		)
-		(property "Value" "4.7u"
+		(property "Value" "3.3u"
 			(at 38.608 50.292 0)
 			(show_name no)
@@
 			)
 		)
-		(property "Value" "4.7u"
+		(property "Value" "3.3u"
 			(at 38.608 121.412 0)
 			(show_name no)
