File: smol-FC-G474-REV-A/sens&IC.kicad_sch (KiCad schematic)
At the start: 24 parts, among them U3 AT7456E, U4 ICM-42688-P, U5 DPS368XTSA1, U6 W25Q128JVSIQ, Y2 27MHz

Commit message: In progress PCB layout
Parts:
- C17: renamed from C23; value 2u2 -> 2.2u
- R14: renamed from R15; value 4.7K -> 4.7k
- R15: renamed from R16; value 4.7K -> 4.7k
- renumbered C17 to C14, C16 to C15, C15 to C16, C24 to C18, C25 to C19, C18 to C20, C19 to C23, C20 to C24, C28 to C25, C27 to C26, C26 to C27, R13 to R11, R14 to R12, R17 to R13, U4 to U3, U3 to U4, U6 to U5, U5 to U6
Connections:
- net GND: no longer U4.29 (EP)
- no-connect marks 6 -> 7

Commit message: Opis Twoich zmian
Connections:
- net V_OUT: now reaches C21.2, C22.2, R12.1
Changed lines of the file:
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@@
+	)
+	(junction
+		(at 128.27 68.58)
+		(diameter 0)
+		(color 0 0 0 0)
 	)
 	(junction
@@
 	(junction
 		(at 57.15 36.83)
-		(diameter 0)
-		(color 0 0 0 0)
-	)
-	(junction
-		(at 128.27 68.58)
 		(diameter 0)
 		(color 0 0 0 0)
@@
 	(wire
 		(pts
+			(xy 128.27 68.58) (xy 124.46 68.58)
+		)
+		(stroke
+			(width 0)
+			(type default)
+		)
+	)
+	(wire
+		(pts
 			(xy 83.82 38.1) (xy 81.28 38.1)
 		)
@@
 	(wire
 		(pts
+			(xy 128.27 68.58) (xy 132.08 68.58)
+		)
+		(stroke
+			(width 0)
+			(type default)
+		)
+	)
+	(wire
+		(pts
 			(xy 231.14 80.01) (xy 228.6 80.01)
 		)
@@
 	(wire
 		(pts
-			(xy 124.46 68.58) (xy 128.27 68.58)
-		)
-		(stroke
-			(width 0)
-			(type default)
-		)
-	)
-	(wire
-		(pts
 			(xy 210.82 22.86) (xy 210.82 26.67)
 		)
@@
 		(pts
 			(xy 34.29 100.33) (xy 34.29 105.41)
-		)
-		(stroke
-			(width 0)
-			(type default)
-		)
-	)
-	(wire
-		(pts
-			(xy 128.27 68.58) (xy 132.08 68.58)
 		)
 		(stroke
@@
 			)
 			(justify left bottom)
+		)
+	)
+	(label "V_OUT"
+		(at 129.54 68.58 0)
+		(effects
+			(font
+				(size 0.508 0.508)
+			)
+			(justify left bottom)
